File: Hardware/TestJig/Jig-Lower-Layer.brd (EAGLE design)
At the start: 63.5 x 54.6 mm, 17 parts, among them J5 CONN_011, J6 SPI, J7 CONN_021, J8 CONN_021

Commit message: fixed white wires on lower layer, added pass throughs for pogo
replaced white wires with bottom traces. 3  traces:  A4, A5, CS

added PTH holes with 1.45mm diameter, giving .15mm clearance of the pogo pin head.

removed cutouts so PCBs can be fabricated
Parts:
- moved S2 141.2 mm to (69.8, 72.4)
Routing:
- net SCL/SCK/RX: track 73.4 -> 102.6 mm
- net !CS: track 0.00 -> 20.1 mm
- net SDA/MISO/TX: track 111.4 -> 110.2 mm
Changed lines of the file:
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@@
 <element name="D1" library="SparkFun-LED" package="LED_5MM" value="" x="12.7" y="50.8"/>
 <element name="U$1" library="Pogo-Footprints" package="1X04" value="CONN_041" x="26.67" y="11.43"/>
-<element name="S2" library="SparkFun-Switches" package="TACTILE_SWITCH_PTH_12MM" value="RST" x="-24.13" y="-33.02">
-<attribute name="PROD_ID" value="SWCH-09185" x="-24.13" y="-33.02" size="1.778" layer="27" font="vector" ratio="15" display="off"/>
-<attribute name="SF_SKU" value="COM-09190" x="-24.13" y="-33.02" size="1.778" layer="27" font="vector" ratio="15" display="off"/>
+<element name="S2" library="SparkFun-Switches" package="TACTILE_SWITCH_PTH_12MM" value="RST" x="69.85" y="72.39">
+<attribute name="PROD_ID" value="SWCH-09185" x="69.85" y="72.39" size="1.778" layer="27" font="vector" ratio="15" display="off"/>
+<attribute name="SF_SKU" value="COM-09190" x="69.85" y="72.39" size="1.778" layer="27" font="vector" ratio="15" display="off"/>
 </element>
 </elements>
@@
 <wire x1="26.67" y1="11.43" x2="26.67" y2="26.67" width="0.254" layer="1"/>
 <contactref element="S2" pad="1"/>
-<wire x1="26.67" y1="11.43" x2="-17.88" y2="-35.52" width="0" layer="19" extent="1-1"/>
+<wire x1="53.34" y1="41.91" x2="76.1" y2="69.89" width="0" layer="19" extent="1-1"/>
 </signal>
 <signal name="ADR/MOSI">
@@
 <contactref element="J6" pad="6"/>
 <contactref element="B1" pad="D10"/>
-<wire x1="34.29" y1="34.29" x2="53.34" y2="31.75" width="0" layer="19" extent="1-1"/>
+<wire x1="53.34" y1="31.75" x2="36.83" y2="31.75" width="0.254" layer="16"/>
+<wire x1="36.83" y1="31.75" x2="34.29" y2="34.29" width="0.254" layer="16"/>
 </signal>
 <signal name="!INT">
@@
 <contactref element="B1" pad="SCL"/>
 <contactref element="B1" pad="D13"/>
-<wire x1="36.83" y1="7.62" x2="34.29" y2="10.16" width="0.254" layer="1"/>
 <wire x1="53.34" y1="39.37" x2="29.21" y2="39.37" width="0.254" layer="1"/>
 <wire x1="29.21" y1="39.37" x2="26.67" y2="36.83" width="0.254" layer="1"/>
@@
 <wire x1="54.991" y1="41.021" x2="53.34" y2="39.37" width="0.254" layer="1"/>
 <contactref element="U$1" pad="4"/>
-<wire x1="34.29" y1="10.16" x2="34.29" y2="11.43" width="0.254" layer="1"/>
 <wire x1="34.29" y1="15.24" x2="34.29" y2="11.43" width="0.254" layer="1"/>
 <contactref element="B1" pad="A5"/>
-<wire x1="5.08" y1="5.08" x2="31.75" y2="17.78" width="0" layer="19" extent="1-1"/>
+<wire x1="5.08" y1="5.08" x2="31.75" y2="5.08" width="0.254" layer="16"/>
+<wire x1="31.75" y1="5.08" x2="34.29" y2="7.62" width="0.254" layer="16"/>
+<wire x1="34.29" y1="7.62" x2="34.29" y2="11.43" width="0.254" layer="16"/>
 </signal>
 <signal name="SDA/MISO/TX">
@@
 <contactref element="B1" pad="SDA"/>
 <contactref element="B1" pad="D12"/>
-<wire x1="36.83" y1="5.08" x2="31.75" y2="10.16" width="0.254" layer="1"/>
 <wire x1="29.21" y1="35.56" x2="29.21" y2="34.29" width="0.254" layer="1"/>
 <wire x1="29.21" y1="34.29" x2="34.29" y2="29.21" width="0.254" layer="1"/>
@@
 <wire x1="52.07" y1="38.1" x2="31.75" y2="38.1" width="0.254" layer="1"/>
 <wire x1="31.75" y1="38.1" x2="29.21" y2="35.56" width="0.254" layer="1"/>
-<wire x1="34.29" y1="29.21" x2="34.29" y2="17.78" width="0.254" layer="1"/>
-<wire x1="34.29" y1="17.78" x2="35.56" y2="16.51" width="0.254" layer="1"/>
-<wire x1="35.56" y1="16.51" x2="35.56" y2="10.16" width="0.254" layer="1"/>
-<wire x1="35.56" y1="10.16" x2="36.83" y2="8.89" width="0.254" layer="1"/>
-<wire x1="36.83" y1="8.89" x2="54.356" y2="8.89" width="0.254" layer="1"/>
-<wire x1="54.356" y1="8.89" x2="54.991" y2="8.255" width="0.254" layer="1"/>
-<wire x1="54.991" y1="8.255" x2="54.991" y2="6.731" width="0.254" layer="1"/>
 <wire x1="53.34" y1="46.99" x2="52.07" y2="46.99" width="0.254" layer="1"/>
 <wire x1="52.07" y1="46.99" x2="50.8" y2="48.26" width="0.254" layer="1"/>
@@
 <wire x1="54.61" y1="36.83" x2="53.34" y2="36.83" width="0.254" layer="1"/>
 <contactref element="U$1" pad="3"/>
-<wire x1="31.75" y1="10.16" x2="31.75" y2="11.43" width="0.254" layer="1"/>
 <contactref element="B1" pad="A4"/>
-<wire x1="36.83" y1="5.08" x2="36.83" y2="8.89" width="0" layer="19" extent="1-1"/>
-<wire x1="5.08" y1="7.62" x2="31.75" y2="10.16" width="0" layer="19" extent="1-1"/>
+<wire x1="5.08" y1="7.62" x2="30.48" y2="7.62" width="0.254" layer="16"/>
+<wire x1="30.48" y1="7.62" x2="31.75" y2="8.89" width="0.254" layer="16"/>
+<wire x1="31.75" y1="8.89" x2="31.75" y2="11.43" width="0.254" layer="16"/>
+<wire x1="34.29" y1="29.21" x2="34.29" y2="19.05" width="0.254" layer="16"/>
+<wire x1="34.29" y1="19.05" x2="31.75" y2="16.51" width="0.254" layer="16"/>
+<wire x1="31.75" y1="16.51" x2="31.75" y2="11.43" width="0.254" layer="16"/>
 </signal>
 <signal name="!RST">
@@
 <contactref element="B1" pad="RES"/>
 <contactref element="S2" pad="3"/>
-<wire x1="5.08" y1="35.56" x2="-17.88" y2="-30.52" width="0" layer="19" extent="1-1"/>
+<wire x1="5.08" y1="35.56" x2="76.1" y2="74.89" width="0" layer="19" extent="1-1"/>
 </signal>
 </signals>
